File: FlexROM_100.sch (KiCad schematic (older format))
At the start: 5 parts, among them J1 LH535618 DIP LEGS, U1 28C256

Commit message: footprint name changed
Parts:
- J1: footprint 000_LOCAL:DIP-28_W15.24mm_pcb_sil_pins -> 000_LOCAL:DIP28_0.6_pcb_sil_pins
Changed lines of the file:
@@
 F 0 "J1" H 4440 4190 50  0000 C CNN
 F 1 "LH535618 DIP LEGS" H 4260 4420 50  0000 C CNN
-F 2 "000_LOCAL:DIP-28_W15.24mm_pcb_sil_pins" H 4260 3040 50  0001 C CNN
+F 2 "000_LOCAL:DIP28_0.6_pcb_sil_pins" H 4260 3040 50  0001 C CNN
 F 3 "http://ww1.microchip.com/downloads/en/DeviceDoc/doc0014.pdf" H 4260 3040 50  0001 C CNN
 	1    4260 3040
