File: uPD23C1000_FLASH.sch (KiCad schematic (older format))
At the start: 7 parts, among them J1 uPD23C1000, J2 Conn_1x2, J3 Conn_1x3, U1 GLS29EE010 (TSOP), U2 SST39SF010 (TSOP), U3 SST39SF010 / GLS29EE010 (PLCC)

Commit message: 27C256_28C256: add jumpers to allow programming without needing a test clip
Other:
- note added: "7x9pin PLCC32"
- note added: "8x14mm TSOP32"
- note added: "8x20mm TSOP32"
- note added: "DIP28 legs"
Changed lines of the file:
@@
 Wire Bus Line
 	1140 2050 1140 5660
+Text Notes 1780 1700 0    50   ~ 0
+DIP28 legs
+Text Notes 4250 1680 0    50   ~ 0
+8x20mm TSOP32
+Text Notes 6270 1700 0    50   ~ 0
+8x14mm TSOP32
+Text Notes 8360 1720 0    50   ~ 0
+7x9pin PLCC32
 $EndSCHEMATC

Commit message: footprint name changed
Parts:
- J1: footprint 000_LOCAL:DIP-28_W15.24mm_pcb_sil_pins -> 000_LOCAL:DIP28_0.6_pcb_sil_pins
Changed lines of the file:
@@
 F 0 "J1" H 2050 4620 50  0000 C CNN
 F 1 "uPD23C1000" H 2050 4510 50  0000 C CNN
-F 2 "000_LOCAL:DIP-28_W15.24mm_pcb_sil_pins" H 2060 3250 50  0001 C CNN
+F 2 "000_LOCAL:DIP28_0.6_pcb_sil_pins" H 2060 3250 50  0001 C CNN
 F 3 "http://ww1.microchip.com/downloads/en/DeviceDoc/doc0014.pdf" H 2060 3250 50  0001 C CNN
 	1    2060 3250
@@
 Wire Bus Line
 	5520 5660 5770 5660
-Wire Bus Line
-	5520 2200 5520 5660
-Wire Bus Line
-	2780 2250 2780 5660
-Wire Bus Line
-	7540 2200 7540 5660
-Wire Bus Line
-	9550 2200 9550 5660
-Wire Bus Line
-	3750 2050 3750 5660
-Wire Bus Line
-	5770 2050 5770 5660
-Wire Bus Line
-	7780 2050 7780 5660
-Wire Bus Line
-	1140 2050 1140 5660
 Text Notes 1780 1700 0    50   ~ 0
 DIP28 legs
@@
 Text Notes 8360 1720 0    50   ~ 0
 7x9pin PLCC32
+Wire Bus Line
+	5520 2200 5520 5660
+Wire Bus Line
+	2780 2250 2780 5660
+Wire Bus Line
+	7540 2200 7540 5660
+Wire Bus Line
+	9550 2200 9550 5660
+Wire Bus Line
+	3750 2050 3750 5660
+Wire Bus Line
+	5770 2050 5770 5660
+Wire Bus Line
+	7780 2050 7780 5660
+Wire Bus Line
+	1140 2050 1140 5660
 $EndSCHEMATC
