File: uPD23C1000_FLASH_DIP32.kicad_pcb (KiCad board)
At the start: 2 copper layers, 16.4 x 39.3 mm, 7 parts, among them J1 uPD23C1000 / FLASH, U1 GLS29EE010 (TSOP), U2 SST39SF010 (TSOP), U3 SST39SF010 / GLS29EE010 (PLCC)

Commit message: readme and silkscreen
Other:
- board text added: "39SF010"
- board text added: "Configure programmer for PLCC version of chip (even if chip is TSOP)"
- board text added: "Place board in programmer ZIF socket"
- board text removed: "Configure programmer for PLCC or DIP version of chip (even if chip is TSOP)"
- board text removed: "GLS29EE010"
- board text removed: "SST39SF010"
- board text removed: "TSOP or PLCC"
Changed lines of the file:
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@@
   (general
     (thickness 1.6)
-    (drawings 25)
+    (drawings 23)
     (tracks 367)
     (zones 0)
@@
   (page A4)
   (layers
-    (0 F.Cu signal hide)
-    (31 B.Cu signal hide)
+    (0 F.Cu signal)
+    (31 B.Cu signal)
     (32 B.Adhes user hide)
     (33 F.Adhes user hide)
     (34 B.Paste user hide)
     (35 F.Paste user hide)
-    (36 B.SilkS user hide)
+    (36 B.SilkS user)
     (37 F.SilkS user)
-    (38 B.Mask user)
+    (38 B.Mask user hide)
     (39 F.Mask user hide)
     (40 Dwgs.User user hide)
@@
     (add_net /~OE)
     (add_net /~WE)
-    (add_net "Net-(J1-Pad1)")
-    (add_net "Net-(U1-Pad6)")
-    (add_net "Net-(U1-Pad9)")
-    (add_net "Net-(U2-Pad6)")
-    (add_net "Net-(U2-Pad9)")
-    (add_net "Net-(U3-Pad1)")
-    (add_net "Net-(U3-Pad30)")
   )
   (module 000_LOCAL:DIP32_0.6_pcb_sil_pins (layer F.Cu)
@@
     )
   )
+  (gr_text 39SF010 (at 150.025 97.875 -90) (layer F.SilkS)
+    (effects (font (size 0.8 0.8) (thickness 0.1)))
+  )
+  (gr_text "Place board in programmer ZIF socket" (at 148.59 80.01 90) (layer B.SilkS)
+    (effects (font (size 0.6 0.6) (thickness 0.08)) (justify left mirror))
+  )
   (gr_text PROGRAMMER (at 151.6253 78.4225) (layer F.SilkS)
     (effects (font (size 0.4572 0.4572) (thickness 0.04064)) (justify left))
   )
-  (gr_text uPD23C1000 (at 143.1036 83.4136) (layer F.SilkS)
-    (effects (font (size 0.4572 0.4572) (thickness 0.04064)) (justify left))
-  )
-  (gr_text GLS29EE010 (at 143.0274 78.7273) (layer F.SilkS)
+  (gr_text uPD23C1000 (at 143.2179 83.4898) (layer F.SilkS)
     (effects (font (size 0.4572 0.4572) (thickness 0.04064)) (justify left))
   )
@@
     (effects (font (size 0.4572 0.4572) (thickness 0.04064)) (justify left))
   )
-  (gr_text SST39SF010 (at 143.0401 78.1812) (layer F.SilkS)
+  (gr_text 39SF010 (at 143.256 78.4098) (layer F.SilkS)
     (effects (font (size 0.4572 0.4572) (thickness 0.04064)) (justify left))
   )
@@
     (effects (font (size 0.8 0.8) (thickness 0.14732)))
   )
-  (gr_text "TSOP or PLCC" (at 148.75 98.95 -90) (layer F.SilkS)
-    (effects (font (size 0.6 0.6) (thickness 0.08)))
-  )
   (gr_text http://tandy.wiki/FlashROM_8300 (at 155.702 93.6625 90) (layer B.SilkS)
     (effects (font (size 0.8 0.8) (thickness 0.1)) (justify mirror))
@@
     (effects (font (size 0.6 0.6) (thickness 0.08)) (justify left mirror))
   )
-  (gr_text GLS29EE010 (at 150 98.95 -90) (layer F.SilkS)
-    (effects (font (size 0.8 0.8) (thickness 0.1)))
-  )
-  (gr_text SST39SF010 (at 151.2 98.95 -90) (layer F.SilkS)
-    (effects (font (size 0.8 0.8) (thickness 0.1)))
-  )
-  (gr_text "Configure programmer for PLCC or DIP version of chip (even if chip is TSOP)" (at 148.59 80.01 90) (layer B.SilkS)
+  (gr_text "Configure programmer for PLCC version of chip (even if chip is TSOP)" (at 149.86 80.01 90) (layer B.SilkS)
     (effects (font (size 0.6 0.6) (thickness 0.08)) (justify left mirror))
   )
