File: uPD23C1000_FLASH_DIP32.kicad_pcb (KiCad board)
At the start: 2 copper layers, 16.4 x 39.3 mm, 7 parts, among them J1 uPD23C1000 / FLASH, U1 GLS29EE010 (TSOP), U2 SST39SF010 (TSOP), U3 SST39SF010 / GLS29EE010 (PLCC)

Commit message: docs for FlashROM_8300, add VPP & pullup on FlashROM_8300 to support old flash, eeprom, & eprom devices.
Parts:
- added R3: 47K, 000_LOCAL:R_0805, F.Cu at (146.1, 80.0)
Connections:
- J1 pad 1: (no net) -> /VPP
- U1 pad 9: (no net) -> /VPP
- U2 pad 9: (no net) -> /VPP
- U3 pad 1: (no net) -> /VPP
Routing:
- net /VPP: track 0.00 -> 23.6 mm, vias 0 -> 1
- net /VCC: track 32.6 -> 43.2 mm
Changed lines of the file:
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@@
     (thickness 1.6)
     (drawings 23)
-    (tracks 367)
+    (tracks 383)
     (zones 0)
-    (modules 7)
-    (nets 32)
+    (modules 8)
+    (nets 33)
   )
   (page A4)
@@
   )
   (setup
-    (last_trace_width 0.25)
+    (last_trace_width 0.18)
     (user_trace_width 0.16)
     (user_trace_width 0.18)
@@
   (net 30 /GND)
   (net 31 /A16_~OE)
+  (net 32 /VPP)
   (net_class Default "This is the default net class."
     (clearance 0.2)
@@
     (add_net /GND)
     (add_net /VCC)
+    (add_net /VPP)
     (add_net /~CE)
     (add_net /~OE)
     (add_net /~WE)
+    (add_net "Net-(U1-Pad6)")
+    (add_net "Net-(U2-Pad6)")
+    (add_net "Net-(U3-Pad30)")
+  )
+  (module 000_LOCAL:R_0805 (layer F.Cu)
+    (at 146.05 80.01)
+    (descr "Resistor SMD 0805, reflow soldering, Vishay (see dcrcw.pdf)")
+    (tags "resistor 0805")
+    (attr smd)
+    (fp_text reference R3 (at -0.0508 -0.0127 -90) (layer F.SilkS)
+      (effects (font (size 0.8 0.8) (thickness 0.1)))
+    )
+    (fp_text value 47K (at 0 1.75) (layer F.Fab)
+      (effects (font (size 1 1) (thickness 0.15)))
+    )
+    (fp_text user %R (at 0 0) (layer F.Fab)
+      (effects (font (size 0.5 0.5) (thickness 0.075)))
+    )
+    (fp_line (start -1 0.62) (end -1 -0.62) (layer F.Fab) (width 0.1))
+    (fp_line (start 1 0.62) (end -1 0.62) (layer F.Fab) (width 0.1))
+    (fp_line (start 1 -0.62) (end 1 0.62) (layer F.Fab) (width 0.1))
+    (fp_line (start -1 -0.62) (end 1 -0.62) (layer F.Fab) (width 0.1))
+    (fp_line (start 0.6 0.88) (end -0.6 0.88) (layer F.SilkS) (width 0.12))
+    (fp_line (start -0.6 -0.88) (end 0.6 -0.88) (layer F.SilkS) (width 0.12))
+    (fp_line (start -1.55 -0.9) (end 1.55 -0.9) (layer F.CrtYd) (width 0.05))
+    (fp_line (start -1.55 -0.9) (end -1.55 0.9) (layer F.CrtYd) (width 0.05))
+    (fp_line (start 1.55 0.9) (end 1.55 -0.9) (layer F.CrtYd) (width 0.05))
+    (fp_line (start 1.55 0.9) (end -1.55 0.9) (layer F.CrtYd) (width 0.05))
+    (pad 1 smd rect (at -0.95 0) (size 0.7 1.3) (layers F.Cu F.Paste F.Mask)
+      (net 32 /VPP))
+    (pad 2 smd rect (at 0.95 0) (size 0.7 1.3) (layers F.Cu F.Paste F.Mask)
+      (net 29 /VCC))
+    (model ${KIPRJMOD}/000_LOCAL.pretty/packages3d/R_0805_2012Metric.step
+      (at (xyz 0 0 0))
+      (scale (xyz 1 1 1))
+      (rotate (xyz 0 0 0))
+    )
   )
   (module 000_LOCAL:PLCC32_7x9 (layer F.Cu)
@@
     (pad 2 smd roundrect (at -1.27 -6.8375) (size 0.6 1.475) (layers F.Cu F.Paste F.Mask) (roundrect_rratio 0.25)
       (net 27 /A16))
-    (pad 1 smd roundrect (at 0 -6.8375) (size 0.6 1.475) (layers F.Cu F.Paste F.Mask) (roundrect_rratio 0.25))
+    (pad 1 smd roundrect (at 0 -6.8375) (size 0.6 1.475) (layers F.Cu F.Paste F.Mask) (roundrect_rratio 0.25)
+      (net 32 /VPP))
     (model ${KIPRJMOD}/000_LOCAL.pretty/packages3d/PLCC32_7x9.step
       (offset (xyz 0 0 0.2))
@@
     (pad 8 smd roundrect (at -0.2401 9.75 180) (size 0.3 1) (layers F.Cu F.Paste F.Mask) (roundrect_rratio 0.25)
       (net 29 /VCC))
-    (pad 9 smd roundrect (at 0.2425 9.75 180) (size 0.3 1) (layers F.Cu F.Paste F.Mask) (roundrect_rratio 0.25))
+    (pad 9 smd roundrect (at 0.2425 9.75 180) (size 0.3 1) (layers F.Cu F.Paste F.Mask) (roundrect_rratio 0.25)
+      (net 32 /VPP))
     (pad 10 smd roundrect (at 0.7505 9.75 180) (size 0.3 1) (layers F.Cu F.Paste F.Mask) (roundrect_rratio 0.25)
       (net 27 /A16))
@@
     (pad 8 smd roundrect (at -0.2401 6.75 180) (size 0.3 1) (layers F.Cu F.Paste F.Mask) (roundrect_rratio 0.25)
       (net 29 /VCC))
-    (pad 9 smd roundrect (at 0.2425 6.75 180) (size 0.3 1) (layers F.Cu F.Paste F.Mask) (roundrect_rratio 0.25))
+    (pad 9 smd roundrect (at 0.2425 6.75 180) (size 0.3 1) (layers F.Cu F.Paste F.Mask) (roundrect_rratio 0.25)
+      (net 32 /VPP))
     (pad 10 smd roundrect (at 0.7505 6.75 180) (size 0.3 1) (layers F.Cu F.Paste F.Mask) (roundrect_rratio 0.25)
       (net 27 /A16))
@@
       (net 30 /GND))
     (pad "" np_thru_hole circle (at 0 -19.65) (size 2 2) (drill 2) (layers *.Cu *.Mask))
-    (pad 1 thru_hole roundrect (at -7.62 -19.05) (size 1.2 1.2) (drill 0.58) (layers *.Cu *.Mask) (roundrect_rratio 0.1))
+    (pad 1 thru_hole roundrect (at -7.62 -19.05) (size 1.2 1.2) (drill 0.58) (layers *.Cu *.Mask) (roundrect_rratio 0.1)
+      (net 32 /VPP))
     (pad 29 thru_hole circle (at 7.62 -11.43) (size 1.2 1.2) (drill 0.58) (layers *.Cu *.Mask)
       (net 1 /A14))
@@
   (segment (start 150.2401 85.7899) (end 157.62 78.41) (width 0.4) (layer B.Cu) (net 29))
   (segment (start 150.2401 87.0721) (end 150.2401 85.7899) (width 0.4) (layer B.Cu) (net 29))
+  (segment (start 155.7526 83.49) (end 155.7526 82.9181) (width 0.18) (layer F.Cu) (net 29))
+  (segment (start 152.8445 80.01) (end 147 80.01) (width 0.18) (layer F.Cu) (net 29))
+  (segment (start 155.7526 82.9181) (end 152.8445 80.01) (width 0.18) (layer F.Cu) (net 29))
   (via (at 148.755 104.7125) (size 0.52) (drill 0.26) (layers F.Cu B.Cu) (net 30))
   (segment (start 148.755 110.135) (end 142.38 116.51) (width 0.4) (layer B.Cu) (net 30))
@@
   (segment (start 155.4 98.45) (end 157.34 98.45) (width 0.18) (layer B.Cu) (net 31))
   (segment (start 151.975 108.915) (end 151.975 101.875) (width 0.18) (layer B.Cu) (net 31))
+  (via (at 150.025 91.0375) (size 0.52) (drill 0.26) (layers F.Cu B.Cu) (net 32))
+  (segment (start 148.59 84.62) (end 142.38 78.41) (width 0.4) (layer B.Cu) (net 32))
+  (segment (start 148.59 87.6808) (end 148.59 84.62) (width 0.4) (layer B.Cu) (net 32))
+  (segment (start 150.025 91.0375) (end 150.025 89.1158) (width 0.4) (layer B.Cu) (net 32))
+  (segment (start 150.025 89.1158) (end 148.59 87.6808) (width 0.4) (layer B.Cu) (net 32))
+  (segment (start 150.025 92.1386) (end 150.025 91.0375) (width 0.3) (layer F.Cu) (net 32))
+  (segment (start 149.7575 93.25) (end 149.7575 92.4061) (width 0.3) (layer F.Cu) (net 32))
+  (segment (start 149.7575 92.4061) (end 150.025 92.1386) (width 0.3) (layer F.Cu) (net 32))
+  (segment (start 149.7575 89) (end 149.7575 89.7627) (width 0.3) (layer F.Cu) (net 32))
+  (segment (start 150.025 90.0302) (end 150.025 91.0375) (width 0.3) (layer F.Cu) (net 32))
+  (segment (start 149.7575 89.7627) (end 150.025 90.0302) (width 0.3) (layer F.Cu) (net 32))
+  (segment (start 143.98 80.01) (end 145.1 80.01) (width 0.18) (layer F.Cu) (net 32))
+  (segment (start 142.38 78.41) (end 143.98 80.01) (width 0.18) (layer F.Cu) (net 32))
 )

Commit message: silkscreen & 3d view
Other:
- board text removed: "PROGRAMMER"
Changed lines of the file:
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@@
   (general
     (thickness 1.6)
-    (drawings 23)
+    (drawings 21)
     (tracks 383)
     (zones 0)
@@
   )
   (setup
-    (last_trace_width 0.18)
+    (last_trace_width 0.25)
     (user_trace_width 0.16)
     (user_trace_width 0.18)
@@
     (add_net /~OE)
     (add_net /~WE)
-    (add_net "Net-(U1-Pad6)")
-    (add_net "Net-(U2-Pad6)")
-    (add_net "Net-(U3-Pad30)")
   )
   (module 000_LOCAL:R_0805 (layer F.Cu)
@@
     (descr "Resistor SMD 0805, reflow soldering, Vishay (see dcrcw.pdf)")
     (tags "resistor 0805")
-    (attr smd)
+    (attr virtual)
     (fp_text reference R3 (at -0.0508 -0.0127 -90) (layer F.SilkS)
       (effects (font (size 0.8 0.8) (thickness 0.1)))
@@
     (effects (font (size 0.6 0.6) (thickness 0.08)) (justify left mirror))
   )
-  (gr_text PROGRAMMER (at 151.6253 78.4225) (layer F.SilkS)
-    (effects (font (size 0.4572 0.4572) (thickness 0.04064)) (justify left))
-  )
   (gr_text uPD23C1000 (at 143.2179 83.4898) (layer F.SilkS)
     (effects (font (size 0.4572 0.4572) (thickness 0.04064)) (justify left))
@@
     (effects (font (size 0.4572 0.4572) (thickness 0.04064)) (justify left))
   )
-  (gr_text 39SF010 (at 143.256 78.4098) (layer F.SilkS)
-    (effects (font (size 0.4572 0.4572) (thickness 0.04064)) (justify left))
-  )
