File: FlexROM_100_programming_adapter.kicad_pcb (KiCad board)
At the start: 2 copper layers, 16.8 x 34.5 mm, 4 parts, among them J1 LH535618 Socket, J2 ~WE~, U1 28C256 pins to programmer

Commit message: silkscreen
Routing:
- net /~WE: track 5.27 -> 4.53 mm
- net /A11: track 11.7 -> 11.0 mm
Other:
- board text added: "DIP28_600 socket this side"
- board text added: "FlexROM_100 Programming Adapter"
- board text added: "Two middle rows, pins to programmer this side"
- board text added: "github.com/bkw777/aDIPters"
- board text added: "single pin this side"
- board text added: "tandy.wiki/FlexROM_100"
Changed lines of the file:
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@@
   (general
     (thickness 1.6)
-    (drawings 5)
-    (tracks 61)
+    (drawings 26)
+    (tracks 56)
     (zones 0)
     (modules 4)
@@
       (effects (font (size 1 1) (thickness 0.15)))
     )
+    (fp_line (start -8.382 -17.272) (end -8.382 17.272) (layer F.CrtYd) (width 0.01))
+    (fp_line (start -8.382 17.272) (end 8.382 17.272) (layer F.CrtYd) (width 0.01))
+    (fp_line (start 8.382 17.272) (end 8.382 -17.272) (layer F.CrtYd) (width 0.01))
     (fp_line (start 8.382 -17.272) (end -8.382 -17.272) (layer F.CrtYd) (width 0.01))
-    (fp_line (start 8.382 17.272) (end 8.382 -17.272) (layer F.CrtYd) (width 0.01))
-    (fp_line (start -8.382 17.272) (end 8.382 17.272) (layer F.CrtYd) (width 0.01))
-    (fp_line (start -8.382 -17.272) (end -8.382 17.272) (layer F.CrtYd) (width 0.01))
     (fp_text user %R (at 0 0) (layer F.Fab)
       (effects (font (size 1 1) (thickness 0.15)))
@@
       (effects (font (size 1 1) (thickness 0.15)))
     )
+    (fp_line (start -8.382 -17.272) (end -8.382 17.272) (layer F.CrtYd) (width 0.01))
+    (fp_line (start -8.382 17.272) (end 8.382 17.272) (layer F.CrtYd) (width 0.01))
+    (fp_line (start 8.382 17.272) (end 8.382 -17.272) (layer F.CrtYd) (width 0.01))
     (fp_line (start 8.382 -17.272) (end -8.382 -17.272) (layer F.CrtYd) (width 0.01))
-    (fp_line (start 8.382 17.272) (end 8.382 -17.272) (layer F.CrtYd) (width 0.01))
-    (fp_line (start -8.382 17.272) (end 8.382 17.272) (layer F.CrtYd) (width 0.01))
-    (fp_line (start -8.382 -17.272) (end -8.382 17.272) (layer F.CrtYd) (width 0.01))
     (fp_text user %R (at 0.27 3.12) (layer F.Fab)
       (effects (font (size 1 1) (thickness 0.15)))
@@
     )
   )
+  (gr_text github.com/bkw777/aDIPters (at 148.222 100 -90) (layer F.SilkS)
+    (effects (font (size 1 1) (thickness 0.15)))
+  )
+  (gr_text tandy.wiki/FlexROM_100 (at 151.524 100 90) (layer B.SilkS)
+    (effects (font (size 1 1) (thickness 0.15)) (justify mirror))
+  )
+  (gr_line (start 156.7945 91.11) (end 154.2545 91.11) (layer F.SilkS) (width 0.12))
+  (gr_line (start 156.7945 88.57) (end 156.7945 91.11) (layer F.SilkS) (width 0.12))
+  (gr_line (start 154.2545 88.57) (end 156.7945 88.57) (layer F.SilkS) (width 0.12))
+  (gr_line (start 154.2545 88.57) (end 154.2545 91.11) (layer F.SilkS) (width 0.12))
+  (gr_line (start 155.5372 91.3386) (end 155.8674 91.6688) (layer F.SilkS) (width 0.12))
+  (gr_line (start 155.5372 91.3386) (end 155.207 91.6688) (layer F.SilkS) (width 0.12))
+  (gr_line (start 155.5372 91.3386) (end 155.5372 92.8626) (layer F.SilkS) (width 0.12))
+  (gr_text "single pin this side" (at 155.588 97.587 -90) (layer F.SilkS)
+    (effects (font (size 0.6 0.6) (thickness 0.08)))
+  )
+  (gr_text "DIP28_600 socket this side" (at 143.777 100 -90) (layer F.SilkS)
+    (effects (font (size 0.8 0.8) (thickness 0.1)))
+  )
+  (gr_text "Two middle rows, pins to programmer this side" (at 148.1585 100 90) (layer B.SilkS)
+    (effects (font (size 0.8 0.8) (thickness 0.1)) (justify mirror))
+  )
+  (gr_line (start 144.92 82.855) (end 147.46 82.855) (layer B.SilkS) (width 0.12))
+  (gr_line (start 144.92 117.145) (end 144.92 82.855) (layer B.SilkS) (width 0.12))
+  (gr_line (start 147.46 117.145) (end 144.92 117.145) (layer B.SilkS) (width 0.12))
+  (gr_line (start 147.46 82.855) (end 147.46 117.145) (layer B.SilkS) (width 0.12))
+  (gr_line (start 152.54 82.855) (end 155.08 82.855) (layer B.SilkS) (width 0.12))
+  (gr_line (start 152.54 117.145) (end 152.54 82.855) (layer B.SilkS) (width 0.12))
+  (gr_line (start 155.08 117.145) (end 152.54 117.145) (layer B.SilkS) (width 0.12))
+  (gr_line (start 155.08 82.855) (end 155.08 117.145) (layer B.SilkS) (width 0.12))
+  (gr_text "FlexROM_100 Programming Adapter" (at 150 100 -90) (layer F.SilkS)
+    (effects (font (size 1 1) (thickness 0.15)))
+  )
   (gr_line (start 141.618 117.272) (end 141.618 82.728) (layer Edge.Cuts) (width 0.05))
   (gr_line (start 158.382 82.728) (end 158.382 117.272) (layer Edge.Cuts) (width 0.05))
@@
   (segment (start 142.38 83.49) (end 143.65 84.76) (width 0.3) (layer F.Cu) (net 1))
   (segment (start 153.81 116.51) (end 157.62 116.51) (width 0.18) (layer F.Cu) (net 2))
+  (segment (start 152.54 101.27) (end 153.81 101.27) (width 0.18) (layer F.Cu) (net 3))
   (segment (start 149.365 98.095) (end 152.54 101.27) (width 0.18) (layer F.Cu) (net 3))
   (segment (start 149.365 89.84) (end 149.365 98.095) (width 0.18) (layer F.Cu) (net 3))
   (segment (start 146.825 87.3) (end 149.365 89.84) (width 0.18) (layer F.Cu) (net 3))
-  (segment (start 152.54 101.27) (end 153.81 101.27) (width 0.18) (layer F.Cu) (net 3))
-  (segment (start 144.92 87.3) (end 146.825 87.3) (width 0.18) (layer F.Cu) (net 3))
-  (segment (start 143.65 86.03) (end 144.92 87.3) (width 0.18) (layer F.Cu) (net 3))
-  (segment (start 142.38 86.03) (end 143.65 86.03) (width 0.18) (layer F.Cu) (net 3))
+  (segment (start 143.65 87.3) (end 146.825 87.3) (width 0.18) (layer F.Cu) (net 3))
+  (segment (start 142.38 86.03) (end 143.65 87.3) (width 0.18) (layer F.Cu) (net 3))
   (segment (start 153.81 113.97) (end 157.62 113.97) (width 0.18) (layer F.Cu) (net 4))
   (segment (start 142.38 88.57) (end 146.19 88.57) (width 0.18) (layer F.Cu) (net 5))
@@
   (segment (start 153.81 106.35) (end 157.62 106.35) (width 0.18) (layer F.Cu) (net 10))
   (segment (start 142.38 96.19) (end 146.19 96.19) (width 0.18) (layer F.Cu) (net 11))
-  (segment (start 156.35 103.81) (end 157.62 103.81) (width 0.18) (layer F.Cu) (net 12))
-  (segment (start 155.715 103.175) (end 156.35 103.81) (width 0.18) (layer F.Cu) (net 12))
-  (segment (start 155.715 101.27) (end 155.715 103.175) (width 0.18) (layer F.Cu) (net 12))
+  (segment (start 155.715 101.905) (end 157.62 103.81) (width 0.18) (layer F.Cu) (net 12))
+  (segment (start 155.715 101.27) (end 155.715 101.905) (width 0.18) (layer F.Cu) (net 12))
+  (segment (start 154.445 100) (end 155.715 101.27) (width 0.18) (layer F.Cu) (net 12))
   (segment (start 153.175 100) (end 154.445 100) (width 0.18) (layer F.Cu) (net 12))
-  (segment (start 154.445 100) (end 155.715 101.27) (width 0.18) (layer F.Cu) (net 12))
   (segment (start 152.54 99.365) (end 153.175 100) (width 0.18) (layer F.Cu) (net 12))
   (segment (start 152.54 97.46) (end 152.54 99.365) (width 0.18) (layer F.Cu) (net 12))
@@
   (segment (start 153.81 98.73) (end 155.08 98.73) (width 0.18) (layer F.Cu) (net 14))
   (segment (start 142.38 101.27) (end 146.19 101.27) (width 0.18) (layer F.Cu) (net 15))
-  (segment (start 157.62 98.73) (end 156.35 98.73) (width 0.18) (layer B.Cu) (net 16))
-  (segment (start 156.35 98.73) (end 155.08 97.46) (width 0.18) (layer B.Cu) (net 16))
-  (segment (start 155.08 97.46) (end 153.175 97.46) (width 0.18) (layer B.Cu) (net 16))
-  (segment (start 153.175 97.46) (end 152.54 96.825) (width 0.18) (layer B.Cu) (net 16))
   (segment (start 152.54 89.84) (end 153.81 88.57) (width 0.18) (layer B.Cu) (net 16))
   (segment (start 152.54 96.825) (end 152.54 89.84) (width 0.18) (layer B.Cu) (net 16))
+  (segment (start 153.175 97.46) (end 152.54 96.825) (width 0.18) (layer B.Cu) (net 16))
+  (segment (start 156.35 97.46) (end 153.175 97.46) (width 0.18) (layer B.Cu) (net 16))
+  (segment (start 157.62 98.73) (end 156.35 97.46) (width 0.18) (layer B.Cu) (net 16))
   (segment (start 142.38 103.81) (end 146.19 103.81) (width 0.18) (layer F.Cu) (net 17))
   (segment (start 142.38 106.35) (end 146.19 106.35) (width 0.18) (layer F.Cu) (net 18))
   (segment (start 147.46 86.03) (end 146.19 86.03) (width 0.18) (layer F.Cu) (net 19))
   (segment (start 150.635 89.205) (end 147.46 86.03) (width 0.18) (layer F.Cu) (net 19))
+  (segment (start 150.635 92.38) (end 150.635 89.205) (width 0.18) (layer F.Cu) (net 19))
+  (segment (start 156.35 94.92) (end 153.175 94.92) (width 0.18) (layer F.Cu) (net 19))
   (segment (start 153.175 94.92) (end 150.635 92.38) (width 0.18) (layer F.Cu) (net 19))
-  (segment (start 155.08 94.92) (end 153.175 94.92) (width 0.18) (layer F.Cu) (net 19))
-  (segment (start 150.635 92.38) (end 150.635 89.205) (width 0.18) (layer F.Cu) (net 19))
-  (segment (start 156.35 93.65) (end 155.08 94.92) (width 0.18) (layer F.Cu) (net 19))
-  (segment (start 157.62 93.65) (end 156.35 93.65) (width 0.18) (layer F.Cu) (net 19))
+  (segment (start 157.62 93.65) (end 156.35 94.92) (width 0.18) (layer F.Cu) (net 19))
   (segment (start 142.38 108.89) (end 146.19 108.89) (width 0.18) (layer F.Cu) (net 20))
   (segment (start 153.81 93.65) (end 155.08 93.65) (width 0.18) (layer F.Cu) (net 21))
@@
   (segment (start 147.46 84.76) (end 156.35 84.76) (width 0.18) (layer B.Cu) (net 26))
   (segment (start 146.19 83.49) (end 147.46 84.76) (width 0.18) (layer B.Cu) (net 26))
-  (segment (start 155.5372 86.4872) (end 155.5372 89.84) (width 0.18) (layer F.Cu) (net 27))
-  (segment (start 155.08 86.03) (end 155.5372 86.4872) (width 0.18) (layer F.Cu) (net 27))
-  (segment (start 153.81 86.03) (end 155.08 86.03) (width 0.18) (layer F.Cu) (net 27))
+  (segment (start 155.5372 87.7572) (end 155.5372 89.84) (width 0.18) (layer F.Cu) (net 27))
+  (segment (start 153.81 86.03) (end 155.5372 87.7572) (width 0.18) (layer F.Cu) (net 27))
 )
