File: FlashROM_100.sch (KiCad schematic (older format))
At the start: 5 parts, among them J1 LH535618 DIP LEGS, U1 29F010

Commit message: FlexROM_100 & FlashROM_100 fix ALE/WE
Parts:
- added JP2: Write-Enable, 000_LOCAL:Pin_Header_Angled_1x02_Pitch2.54mm, symbol 000_LOCAL:Jumper_2_Bridged
- JP1: value ~CS~ breakout (REX TP1) -> ~CS~ breakout
Connections:
- net ~WE: now also JP2.1 (A); no longer J1.23 (ALE)
- new net ALE: J1.23 (ALE), JP2.2 (B)
Other:
- moved on the sheet: R1
Changed lines of the file:
@@
 Sheet 1 1
 Title "28C256 SOIC to LH535618 DIP"
-Date ""
+Date "2020-11-23"
 Rev ""
-Comp ""
+Comp "Brian K. White - b.kenyon.w@gmail.com"
 Comment1 "TRS-80 Model 100 system rom M12"
 Comment2 "With REX main ROM support"
@@
 P 3500 4830
 F 0 "JP1" H 3500 4910 50  0000 C CNN
-F 1 "~CS~ breakout (REX TP1)" H 3500 4990 50  0000 C CNN
+F 1 "~CS~ breakout" H 3500 4990 50  0000 C CNN
 F 2 "000_LOCAL:Pin_Header_Angled_1x02_Pitch2.54mm" H 3500 4830 50  0001 C CNN
 F 3 "~" H 3500 4830 50  0001 C CNN
@@
 Wire Bus Line
 	3000 5700 4580 5700
-Entry Wire Line
-	3000 5100 3100 5200
 $Comp
 L 000_LOCAL:R_US R1
 U 1 1 5E6B3AF8
-P 3350 5200
-F 0 "R1" V 3260 5050 50  0000 C CNN
-F 1 "47K" V 3260 5200 50  0000 C CNN
-F 2 "000_LOCAL:R_0805" H 3350 5200 50  0001 C CNN
-F 3 "~" H 3350 5200 50  0001 C CNN
-	1    3350 5200
+P 3850 5300
+F 0 "R1" V 3760 5150 50  0000 C CNN
+F 1 "47K" V 3760 5300 50  0000 C CNN
+F 2 "000_LOCAL:R_0805" H 3850 5300 50  0001 C CNN
+F 3 "~" H 3850 5300 50  0001 C CNN
+	1    3850 5300
 	0    -1   -1   0
 $EndComp
-Text Label 3100 5200 0    50   ~ 0
-~WE
 Wire Wire Line
 	3100 2300 3460 2300
@@
 L power:VCC #PWR0104
 U 1 1 5FAA9518
-P 3500 5200
-F 0 "#PWR0104" H 3500 5050 50  0001 C CNN
-F 1 "VCC" V 3540 5330 50  0000 L CNN
-F 2 "" H 3500 5200 50  0001 C CNN
-F 3 "" H 3500 5200 50  0001 C CNN
-	1    3500 5200
+P 4000 5300
+F 0 "#PWR0104" H 4000 5150 50  0001 C CNN
+F 1 "VCC" V 4040 5430 50  0000 L CNN
+F 2 "" H 4000 5300 50  0001 C CNN
+F 3 "" H 4000 5300 50  0001 C CNN
+	1    4000 5300
 	0    1    1    0
 $EndComp
@@
 	3000 3800 3100 3900
 Text Label 3100 3900 0    50   ~ 0
-~WE
+ALE
 Wire Wire Line
 	3100 3900 3460 3900
@@
 	3100 4930 3700 4930
 Connection ~ 3700 4830
-Wire Wire Line
-	3100 5200 3200 5200
+Entry Wire Line
+	3000 5200 3100 5300
+Entry Wire Line
+	3000 5300 3100 5400
+$Comp
+L 000_LOCAL:Jumper_2_Bridged JP2
+U 1 1 5FBC3795
+P 3500 5300
+F 0 "JP2" H 3500 5380 50  0000 C CNN
+F 1 "Write-Enable" H 3500 5460 50  0000 C CNN
+F 2 "000_LOCAL:Pin_Header_Angled_1x02_Pitch2.54mm" H 3500 5300 50  0001 C CNN
+F 3 "~" H 3500 5300 50  0001 C CNN
+	1    3500 5300
+	-1   0    0    -1
+$EndComp
+Text Label 3100 5300 0    50   ~ 0
+ALE
+Text Label 3100 5400 0    50   ~ 0
+~WE
+Wire Wire Line
+	3700 5300 3700 5400
+Wire Wire Line
+	3100 5300 3300 5300
+Wire Wire Line
+	3100 5400 3700 5400
+Connection ~ 3700 5300
 Wire Bus Line
 	7770 2200 7770 5700

Commit message: simpler programming adapters, update pics and BOMs
Connections:
- net ALE renamed ALE_~WE
- net ~CS_IN renamed ~CS
- net ~CS_OUT renamed ~CS_BUS
Changed lines of the file:
@@
 ~OE
 Text Label 3100 4100 0    50   ~ 0
-~CS_OUT
+~CS_BUS
 Text Label 5900 4600 0    50   ~ 0
 ~OE
 Text Label 5900 4500 0    50   ~ 0
-~CS_IN
+~CS
 Text Label 3100 2400 0    50   ~ 0
 A1
@@
 $EndComp
 Text Label 3100 4830 0    50   ~ 0
-~CS_OUT
+~CS_BUS
 Text Label 3100 4930 0    50   ~ 0
-~CS_IN
+~CS
 Wire Bus Line
 	3000 5700 4580 5700
@@
 	3000 3800 3100 3900
 Text Label 3100 3900 0    50   ~ 0
-ALE
+ALE_~WE
 Wire Wire Line
 	3100 3900 3460 3900
@@
 $EndComp
 Text Label 3100 5300 0    50   ~ 0
-ALE
+ALE_~WE
 Text Label 3100 5400 0    50   ~ 0
 ~WE
