File: FlexROM_100_programming_adapter.sch (KiCad schematic (older format))
At the start: 6 parts, among them J1 LH535618 DIP LEGS, J2 ~WE~, U1 28C256

Commit message: FlexROM_100 programming adapter, FlexROM_102 programming jumpers
Parts:
- removed JP1: ~CS~ breakout (REX TP1), 000_LOCAL:Pin_Header_Angled_1x02_Pitch2.54mm, symbol 000_LOCAL:Jumper_2_Bridged
- removed R1, R2: 47K, 000_LOCAL:R_0805, symbol 000_LOCAL:R_US
- J1: value LH535618 DIP LEGS -> LH535618 Socket; footprint 000_LOCAL:DIP28_0.6_pcb_sil_pins -> 000_LOCAL:DIP28_0.6
- J2: footprint 000_LOCAL:Pin_1x1_hole -> 000_LOCAL:Pin_1x1; symbol 000_LOCAL:Conn_01x01_Female -> 000_LOCAL:Conn_01x01_Male
- U1: value 28C256 -> 28C256 pins to programmer; footprint 000_LOCAL:SOIC28W -> 000_LOCAL:2x28_0.3_0.1_pins
Connections:
- wire segments 65 -> 56
Other:
- note removed: "~WE~ to programming adapter"
Changed lines of the file:
@@
 P 6670 3040
 F 0 "U1" H 6810 4160 50  0000 C CNN
-F 1 "28C256" H 6670 4350 50  0000 C CNN
-F 2 "000_LOCAL:SOIC28W" H 6670 3040 50  0001 C CNN
+F 1 "28C256 pins to programmer" H 6670 4350 50  0000 C CNN
+F 2 "000_LOCAL:2x28_0.3_0.1_pins" H 6670 3040 50  0001 C CNN
 F 3 "http://ww1.microchip.com/downloads/en/DeviceDoc/doc0006.pdf" H 6670 3040 50  0001 C CNN
 	1    6670 3040
@@
 P 4260 3040
 F 0 "J1" H 4440 4190 50  0000 C CNN
-F 1 "LH535618 DIP LEGS" H 4260 4420 50  0000 C CNN
-F 2 "000_LOCAL:DIP28_0.6_pcb_sil_pins" H 4260 3040 50  0001 C CNN
+F 1 "LH535618 Socket" H 4260 4420 50  0000 C CNN
+F 2 "000_LOCAL:DIP28_0.6" H 4260 3040 50  0001 C CNN
 F 3 "http://ww1.microchip.com/downloads/en/DeviceDoc/doc0014.pdf" H 4260 3040 50  0001 C CNN
 	1    4260 3040
@@
 Text Notes 4110 3770 0    50   ~ 0
 (ALE)
-Entry Wire Line
-	3400 4570 3500 4670
-Entry Wire Line
-	3400 4670 3500 4770
+Wire Bus Line
+	3400 5540 4980 5540
+Connection ~ 5830 5540
+Wire Bus Line
+	5830 5540 7400 5540
+Entry Wire Line
+	5830 4400 5930 4500
+Text Label 5930 4500 0    50   ~ 0
+~WE
+Connection ~ 4980 5540
+Wire Bus Line
+	4980 5540 5830 5540
+Wire Bus Line
+	5830 5540 6590 5540
+Wire Wire Line
+	3500 1940 4260 1940
+Wire Wire Line
+	3500 2140 3860 2140
+Wire Wire Line
+	3500 2240 3860 2240
+Wire Wire Line
+	3500 2340 3860 2340
+Wire Wire Line
+	3500 2440 3860 2440
+Wire Wire Line
+	3500 2540 3860 2540
+Wire Wire Line
+	3500 2640 3860 2640
+Wire Wire Line
+	3500 2740 3860 2740
+Wire Wire Line
+	3500 2840 3860 2840
+Wire Wire Line
+	3500 2940 3860 2940
+Wire Wire Line
+	3500 3040 3860 3040
+Wire Wire Line
+	3500 3140 3860 3140
+Wire Wire Line
+	3500 3240 3860 3240
+Wire Wire Line
+	3500 3340 3860 3340
+Wire Wire Line
+	3500 3440 3860 3440
+Wire Wire Line
+	3500 3540 3860 3540
+Wire Wire Line
+	3500 3840 3860 3840
+Wire Wire Line
+	3500 3940 3860 3940
+Wire Wire Line
+	3500 4140 4260 4140
+Wire Wire Line
+	4660 2140 4880 2140
+Wire Wire Line
+	4660 2240 4880 2240
+Wire Wire Line
+	4660 2340 4880 2340
+Wire Wire Line
+	4660 2440 4880 2440
+Wire Wire Line
+	4660 2540 4880 2540
+Wire Wire Line
+	4660 2640 4880 2640
+Wire Wire Line
+	4660 2740 4880 2740
+Wire Wire Line
+	4660 2840 4880 2840
+Wire Wire Line
+	5930 1940 6670 1940
+Wire Wire Line
+	5930 2140 6270 2140
+Wire Wire Line
+	5930 2240 6270 2240
+Wire Wire Line
+	5930 2340 6270 2340
+Wire Wire Line
+	5930 2440 6270 2440
+Wire Wire Line
+	5930 2540 6270 2540
+Wire Wire Line
+	5930 2640 6270 2640
+Wire Wire Line
+	5930 2740 6270 2740
+Wire Wire Line
+	5930 2840 6270 2840
+Wire Wire Line
+	5930 2940 6270 2940
+Wire Wire Line
+	5930 3040 6270 3040
+Wire Wire Line
+	5930 3140 6270 3140
+Wire Wire Line
+	5930 3240 6270 3240
+Wire Wire Line
+	5930 3340 6270 3340
+Wire Wire Line
+	5930 3440 6270 3440
+Wire Wire Line
+	5930 3540 6270 3540
+Wire Wire Line
+	5930 3740 6270 3740
+Wire Wire Line
+	5930 3840 6270 3840
+Wire Wire Line
+	5930 3940 6270 3940
+Wire Wire Line
+	5930 4140 6670 4140
+Wire Wire Line
+	7070 2140 7300 2140
+Wire Wire Line
+	7070 2240 7300 2240
+Wire Wire Line
+	7070 2340 7300 2340
+Wire Wire Line
+	7070 2440 7300 2440
+Wire Wire Line
+	7070 2540 7300 2540
+Wire Wire Line
+	7070 2640 7300 2640
+Wire Wire Line
+	7070 2740 7300 2740
+Wire Wire Line
+	7070 2840 7300 2840
 $Comp
-L 000_LOCAL:Jumper_2_Bridged JP1
-U 1 1 5E68B8A2
-P 4020 4670
-F 0 "JP1" H 4020 4750 50  0000 C CNN
-F 1 "~CS~ breakout (REX TP1)" H 4020 4830 50  0000 C CNN
-F 2 "000_LOCAL:Pin_Header_Angled_1x02_Pitch2.54mm" H 4020 4670 50  0001 C CNN
-F 3 "~" H 4020 4670 50  0001 C CNN
-	1    4020 4670
+L 000_LOCAL:Conn_01x01_Male J2
+U 1 1 5FA33369
+P 6330 4500
+F 0 "J2" H 6230 4500 50  0000 L CNN
+F 1 "~WE~" H 6100 4490 50  0000 L CNN
+F 2 "000_LOCAL:Pin_1x1" H 6330 4500 50  0001 C CNN
+F 3 "~" H 6330 4500 50  0001 C CNN
+	1    6330 4500
 	-1   0    0    -1
 $EndComp
-Entry Wire Line
-	3400 4770 3500 4870
-$Comp
-L 000_LOCAL:R_US R2
-U 1 1 5E68C7F8
-P 4080 4870
-F 0 "R2" V 4040 4550 50  0000 C CNN
-F 1 "47K" V 4040 4700 50  0000 C CNN
-F 2 "000_LOCAL:R_0805" H 4080 4870 50  0001 C CNN
-F 3 "~" H 4080 4870 50  0001 C CNN
-	1    4080 4870
-	0    1    1    0
-$EndComp
-Wire Wire Line
-	3500 4670 3820 4670
-Text Label 3500 4670 0    50   ~ 0
-~CS_OUT
-Wire Wire Line
-	3500 4870 3930 4870
-Text Label 3500 4770 0    50   ~ 0
-~CS_IN
-Text Label 3500 4870 0    50   ~ 0
-VCC
-Wire Bus Line
-	3400 5540 4980 5540
-Connection ~ 5830 5540
-Wire Bus Line
-	5830 5540 7400 5540
-Entry Wire Line
-	3400 5070 3500 5170
-Entry Wire Line
-	3400 5170 3500 5270
-$Comp
-L 000_LOCAL:R_US R1
-U 1 1 5E6B3AF8
-P 4080 5270
-F 0 "R1" V 4040 4940 50  0000 C CNN
-F 1 "47K" V 4040 5100 50  0000 C CNN
-F 2 "000_LOCAL:R_0805" H 4080 5270 50  0001 C CNN
-F 3 "~" H 4080 5270 50  0001 C CNN
-	1    4080 5270
-	0    1    1    0
-$EndComp
-Wire Wire Line
-	3500 5270 3930 5270
-Wire Wire Line
-	4230 5270 4230 5170
-Text Label 3500 5270 0    50   ~ 0
-VCC
-Text Label 3500 5170 0    50   ~ 0
-~WE
-Connection ~ 4980 5540
-Wire Bus Line
-	4980 5540 5830 5540
-Wire Bus Line
-	5830 5540 6590 5540
-Wire Wire Line
-	3500 1940 4260 1940
-Wire Wire Line
-	3500 2140 3860 2140
-Wire Wire Line
-	3500 2240 3860 2240
-Wire Wire Line
-	3500 2340 3860 2340
-Wire Wire Line
-	3500 2440 3860 2440
-Wire Wire Line
-	3500 2540 3860 2540
-Wire Wire Line
-	3500 2640 3860 2640
-Wire Wire Line
-	3500 2740 3860 2740
-Wire Wire Line
-	3500 2840 3860 2840
-Wire Wire Line
-	3500 2940 3860 2940
-Wire Wire Line
-	3500 3040 3860 3040
-Wire Wire Line
-	3500 3140 3860 3140
-Wire Wire Line
-	3500 3240 3860 3240
-Wire Wire Line
-	3500 3340 3860 3340
-Wire Wire Line
-	3500 3440 3860 3440
-Wire Wire Line
-	3500 3540 3860 3540
-Wire Wire Line
-	3500 3840 3860 3840
-Wire Wire Line
-	3500 3940 3860 3940
-Wire Wire Line
-	3500 4140 4260 4140
-Wire Wire Line
-	4660 2140 4880 2140
-Wire Wire Line
-	4660 2240 4880 2240
-Wire Wire Line
-	4660 2340 4880 2340
-Wire Wire Line
-	4660 2440 4880 2440
-Wire Wire Line
-	4660 2540 4880 2540
-Wire Wire Line
-	4660 2640 4880 2640
-Wire Wire Line
-	4660 2740 4880 2740
-Wire Wire Line
-	4660 2840 4880 2840
-Wire Wire Line
-	5930 1940 6670 1940
-Wire Wire Line
-	5930 2140 6270 2140
-Wire Wire Line
-	5930 2240 6270 2240
-Wire Wire Line
-	5930 2340 6270 2340
-Wire Wire Line
-	5930 2440 6270 2440
-Wire Wire Line
-	5930 2540 6270 2540
-Wire Wire Line
-	5930 2640 6270 2640
-Wire Wire Line
-	5930 2740 6270 2740
-Wire Wire Line
-	5930 2840 6270 2840
-Wire Wire Line
-	5930 2940 6270 2940
-Wire Wire Line
-	5930 3040 6270 3040
-Wire Wire Line
-	5930 3140 6270 3140
-Wire Wire Line
-	5930 3240 6270 3240
-Wire Wire Line
-	5930 3340 6270 3340
-Wire Wire Line
-	5930 3440 6270 3440
-Wire Wire Line
-	5930 3540 6270 3540
-Wire Wire Line
-	5930 3740 6270 3740
-Wire Wire Line
-	5930 3840 6270 3840
-Wire Wire Line
-	5930 3940 6270 3940
-Wire Wire Line
-	5930 4140 6670 4140
-Wire Wire Line
-	7070 2140 7300 2140
-Wire Wire Line
-	7070 2240 7300 2240
-Wire Wire Line
-	7070 2340 7300 2340
-Wire Wire Line
-	7070 2440 7300 2440
-Wire Wire Line
-	7070 2540 7300 2540
-Wire Wire Line
-	7070 2640 7300 2640
-Wire Wire Line
-	7070 2740 7300 2740
-Wire Wire Line
-	7070 2840 7300 2840
-Wire Wire Line
-	4360 4670 4360 4770
-Wire Wire Line
-	4230 4870 4360 4870
-Wire Wire Line
-	3500 4770 4360 4770
-Connection ~ 4360 4770
-Wire Wire Line
-	4360 4770 4360 4870
-Wire Wire Line
-	4360 4670 4220 4670
-$Comp
-L 000_LOCAL:Conn_01x01_Female J2
-U 1 1 5FA33369
-P 4430 5170
-F 0 "J2" H 4450 5170 50  0000 L CNN
-F 1 "~WE~" H 4570 5160 50  0000 L CNN
-F 2 "000_LOCAL:Pin_1x1_hole" H 4430 5170 50  0001 C CNN
-F 3 "~" H 4430 5170 50  0001 C CNN
-	1    4430 5170
-	1    0    0    -1
-$EndComp
-Wire Wire Line
-	3500 5170 4230 5170
-Connection ~ 4230 5170
 NoConn ~ 3860 3740
+Wire Wire Line
+	5930 4500 6130 4500
 Wire Bus Line
 	4980 2040 4980 5540
@@
 Wire Bus Line
 	3400 1840 3400 5540
-Text Notes 3890 5090 0    50   ~ 0
-~WE~ to programming adapter
 $EndSCHEMATC

Commit message: Add FlashROM_100. /WE pin on FlexROM_100
Parts:
- removed J2: ~WE~, 000_LOCAL:Pin_1x1, symbol 000_LOCAL:Conn_01x01_Male
- U1: value 28C256 pins to programmer -> 28C256 pinout to programmer
Connections:
- net labels added: ~CE
- net labels removed: ~CS_IN, ~CS_OUT
- no-connect marks 1 -> 0
Other:
- note removed: "(ALE)"
Changed lines of the file:
@@
 P 6670 3040
 F 0 "U1" H 6810 4160 50  0000 C CNN
-F 1 "28C256 pins to programmer" H 6670 4350 50  0000 C CNN
+F 1 "28C256 pinout to programmer" H 6670 4350 50  0000 C CNN
 F 2 "000_LOCAL:2x28_0.3_0.1_pins" H 6670 3040 50  0001 C CNN
 F 3 "http://ww1.microchip.com/downloads/en/DeviceDoc/doc0006.pdf" H 6670 3040 50  0001 C CNN
@@
 ~OE
 Text Label 3500 3940 0    50   ~ 0
-~CS_OUT
+~CE
 Text Label 5930 3840 0    50   ~ 0
 ~OE
 Text Label 5930 3940 0    50   ~ 0
-~CS_IN
+~CE
 Text Label 3500 2240 0    50   ~ 0
 A1
@@
 Text Label 7300 2840 2    50   ~ 0
 D7
-Text Notes 4110 3770 0    50   ~ 0
-(ALE)
 Wire Bus Line
 	3400 5540 4980 5540
@@
 Wire Bus Line
 	5830 5540 7400 5540
-Entry Wire Line
-	5830 4400 5930 4500
-Text Label 5930 4500 0    50   ~ 0
+Connection ~ 4980 5540
+Wire Bus Line
+	4980 5540 5830 5540
+Wire Bus Line
+	5830 5540 6590 5540
+Wire Wire Line
+	3500 1940 4260 1940
+Wire Wire Line
+	3500 2140 3860 2140
+Wire Wire Line
+	3500 2240 3860 2240
+Wire Wire Line
+	3500 2340 3860 2340
+Wire Wire Line
+	3500 2440 3860 2440
+Wire Wire Line
+	3500 2540 3860 2540
+Wire Wire Line
+	3500 2640 3860 2640
+Wire Wire Line
+	3500 2740 3860 2740
+Wire Wire Line
+	3500 2840 3860 2840
+Wire Wire Line
+	3500 2940 3860 2940
+Wire Wire Line
+	3500 3040 3860 3040
+Wire Wire Line
+	3500 3140 3860 3140
+Wire Wire Line
+	3500 3240 3860 3240
+Wire Wire Line
+	3500 3340 3860 3340
+Wire Wire Line
+	3500 3440 3860 3440
+Wire Wire Line
+	3500 3540 3860 3540
+Wire Wire Line
+	3500 3840 3860 3840
+Wire Wire Line
+	3500 3940 3860 3940
+Wire Wire Line
+	3500 4140 4260 4140
+Wire Wire Line
+	4660 2140 4880 2140
+Wire Wire Line
+	4660 2240 4880 2240
+Wire Wire Line
+	4660 2340 4880 2340
+Wire Wire Line
+	4660 2440 4880 2440
+Wire Wire Line
+	4660 2540 4880 2540
+Wire Wire Line
+	4660 2640 4880 2640
+Wire Wire Line
+	4660 2740 4880 2740
+Wire Wire Line
+	4660 2840 4880 2840
+Wire Wire Line
+	5930 1940 6670 1940
+Wire Wire Line
+	5930 2140 6270 2140
+Wire Wire Line
+	5930 2240 6270 2240
+Wire Wire Line
+	5930 2340 6270 2340
+Wire Wire Line
+	5930 2440 6270 2440
+Wire Wire Line
+	5930 2540 6270 2540
+Wire Wire Line
+	5930 2640 6270 2640
+Wire Wire Line
+	5930 2740 6270 2740
+Wire Wire Line
+	5930 2840 6270 2840
+Wire Wire Line
+	5930 2940 6270 2940
+Wire Wire Line
+	5930 3040 6270 3040
+Wire Wire Line
+	5930 3140 6270 3140
+Wire Wire Line
+	5930 3240 6270 3240
+Wire Wire Line
+	5930 3340 6270 3340
+Wire Wire Line
+	5930 3440 6270 3440
+Wire Wire Line
+	5930 3540 6270 3540
+Wire Wire Line
+	5930 3740 6270 3740
+Wire Wire Line
+	5930 3840 6270 3840
+Wire Wire Line
+	5930 3940 6270 3940
+Wire Wire Line
+	5930 4140 6670 4140
+Wire Wire Line
+	7070 2140 7300 2140
+Wire Wire Line
+	7070 2240 7300 2240
+Wire Wire Line
+	7070 2340 7300 2340
+Wire Wire Line
+	7070 2440 7300 2440
+Wire Wire Line
+	7070 2540 7300 2540
+Wire Wire Line
+	7070 2640 7300 2640
+Wire Wire Line
+	7070 2740 7300 2740
+Wire Wire Line
+	7070 2840 7300 2840
+Entry Wire Line
+	3400 3640 3500 3740
+Wire Wire Line
+	3860 3740 3500 3740
+Text Label 3500 3740 0    50   ~ 0
 ~WE
-Connection ~ 4980 5540
-Wire Bus Line
-	4980 5540 5830 5540
-Wire Bus Line
-	5830 5540 6590 5540
-Wire Wire Line
-	3500 1940 4260 1940
-Wire Wire Line
-	3500 2140 3860 2140
-Wire Wire Line
-	3500 2240 3860 2240
-Wire Wire Line
-	3500 2340 3860 2340
-Wire Wire Line
-	3500 2440 3860 2440
-Wire Wire Line
-	3500 2540 3860 2540
-Wire Wire Line
-	3500 2640 3860 2640
-Wire Wire Line
-	3500 2740 3860 2740
-Wire Wire Line
-	3500 2840 3860 2840
-Wire Wire Line
-	3500 2940 3860 2940
-Wire Wire Line
-	3500 3040 3860 3040
-Wire Wire Line
-	3500 3140 3860 3140
-Wire Wire Line
-	3500 3240 3860 3240
-Wire Wire Line
-	3500 3340 3860 3340
-Wire Wire Line
-	3500 3440 3860 3440
-Wire Wire Line
-	3500 3540 3860 3540
-Wire Wire Line
-	3500 3840 3860 3840
-Wire Wire Line
-	3500 3940 3860 3940
-Wire Wire Line
-	3500 4140 4260 4140
-Wire Wire Line
-	4660 2140 4880 2140
-Wire Wire Line
-	4660 2240 4880 2240
-Wire Wire Line
-	4660 2340 4880 2340
-Wire Wire Line
-	4660 2440 4880 2440
-Wire Wire Line
-	4660 2540 4880 2540
-Wire Wire Line
-	4660 2640 4880 2640
-Wire Wire Line
-	4660 2740 4880 2740
-Wire Wire Line
-	4660 2840 4880 2840
-Wire Wire Line
-	5930 1940 6670 1940
-Wire Wire Line
-	5930 2140 6270 2140
-Wire Wire Line
-	5930 2240 6270 2240
-Wire Wire Line
-	5930 2340 6270 2340
-Wire Wire Line
-	5930 2440 6270 2440
-Wire Wire Line
-	5930 2540 6270 2540
-Wire Wire Line
-	5930 2640 6270 2640
-Wire Wire Line
-	5930 2740 6270 2740
-Wire Wire Line
-	5930 2840 6270 2840
-Wire Wire Line
-	5930 2940 6270 2940
-Wire Wire Line
-	5930 3040 6270 3040
-Wire Wire Line
-	5930 3140 6270 3140
-Wire Wire Line
-	5930 3240 6270 3240
-Wire Wire Line
-	5930 3340 6270 3340
-Wire Wire Line
-	5930 3440 6270 3440
-Wire Wire Line
-	5930 3540 6270 3540
-Wire Wire Line
-	5930 3740 6270 3740
-Wire Wire Line
-	5930 3840 6270 3840
-Wire Wire Line
-	5930 3940 6270 3940
-Wire Wire Line
-	5930 4140 6670 4140
-Wire Wire Line
-	7070 2140 7300 2140
-Wire Wire Line
-	7070 2240 7300 2240
-Wire Wire Line
-	7070 2340 7300 2340
-Wire Wire Line
-	7070 2440 7300 2440
-Wire Wire Line
-	7070 2540 7300 2540
-Wire Wire Line
-	7070 2640 7300 2640
-Wire Wire Line
-	7070 2740 7300 2740
-Wire Wire Line
-	7070 2840 7300 2840
-$Comp
-L 000_LOCAL:Conn_01x01_Male J2
-U 1 1 5FA33369
-P 6330 4500
-F 0 "J2" H 6230 4500 50  0000 L CNN
-F 1 "~WE~" H 6100 4490 50  0000 L CNN
-F 2 "000_LOCAL:Pin_1x1" H 6330 4500 50  0001 C CNN
-F 3 "~" H 6330 4500 50  0001 C CNN
-	1    6330 4500
-	-1   0    0    -1
-$EndComp
-NoConn ~ 3860 3740
-Wire Wire Line
-	5930 4500 6130 4500
 Wire Bus Line
 	4980 2040 4980 5540
