File: FlashROM_100_PLCC.sch (KiCad schematic (older format))
At the start: 6 parts, among them J1 LH535618 DIP LEGS, U1 29F010

Commit message: add model 100 optrom programming adapter. readme and renders
Parts:
- U1: footprint 000_LOCAL:TSOP32-14mm -> 000_LOCAL:PLCC32_7x9
Changed lines of the file:
@@
 F 0 "U1" H 6840 3500 50  0000 C CNN
 F 1 "29F010" H 6840 5150 50  0000 C CNN
-F 2 "000_LOCAL:TSOP32-14mm" H 6840 3500 50  0001 C CNN
+F 2 "000_LOCAL:PLCC32_7x9" H 6840 3500 50  0001 C CNN
 F 3 "http://ww1.microchip.com/downloads/en/DeviceDoc/doc0006.pdf" H 6840 3500 50  0001 C CNN
 	1    6840 3500
