File: FlashROM_100_TSOP.kicad_pcb (KiCad board)
At the start: 2 copper layers, 35.6 x 17.8 mm, 6 parts, among them J1 LH535618 DIP LEGS, U1 29F010

Commit message: minor touches
Parts:
- R1, R2: value 47K -> 100K
Connections:
- net /~{CS} renamed /~{CS_IC}
Routing:
- net /~{CS_BUS}: track 2.92 -> 2.29 mm
Other:
- board text added: "BUS"
- board text added: "IC"
- board text added: "REX_Classic main ROM support: ~{CS_BUS} to REX TP1 to boot REX main rom ~{CS_BUS} to ~{CS_IC} to boot internal main rom"
- board text removed: "IN"
- board text removed: "OUT"
- board text removed: "REX_Classic main ROM support: ~{CS}_OUT to REX TP1 to boot REX main rom ~{CS}_OUT to ~{CS}_IN to boot internal main rom"
